Commit message: Added velocity controller

File: urdf/kobuki_description.urdf.xacro (robot description, xacro)
@@ -1,4 +1,5 @@
 <?xml version="1.0" ?>
 <robot name="kobuki" xmlns:xacro="http://ros.org/wiki/xacro">
+  <xacro:arg name="robot_namespace" default="/" />
   <!-- Include Parameters -->
   <xacro:include filename="$(find kobuki_pkg)/urdf/kobuki_parameters.urdf.xacro"/>
@@ -29,12 +30,9 @@
   />
   <!-- Left Traction Wheel -->
-  <joint name="wheel_left_joint" type="continuous">
-    <parent link="base_link"/>
-    <child link="wheel_left_link"/>
-    <origin xyz="0.00 ${0.23/2} 0.0250" rpy="${-M_PI/2} 0 0"/>
-    <axis xyz="0 0 1"/>
-  </joint>
-  <link_wheel_kobuki
-    name="wheel_left_link"
+  <wheel_kobuki
+    name="wheel_left"
+    joint_origin_xyz="0.00 ${0.23/2} 0.0250"
+    joint_origin_rpy="${-M_PI/2} 0 0"
+    joint_axis_xyz="0 0 1"
     visual_rpy="0 0 0"
     visual_xyz="0 0 0"
@@ -51,12 +49,9 @@
   />
   <!-- Right Traction Wheel -->
-  <joint name="wheel_right_joint" type="continuous">
-    <parent link="base_link"/>
-    <child link="wheel_right_link"/>
-    <origin xyz="0.00 -${0.23/2} 0.0250" rpy="${-M_PI/2} 0 0"/>
-    <axis xyz="0 0 1"/>
-  </joint>
-  <link_wheel_kobuki
-    name="wheel_right_link"
+   <wheel_kobuki
+    name="wheel_right"
+    joint_origin_xyz="0.00 -${0.23/2} 0.0250"
+    joint_origin_rpy="${-M_PI/2} 0 0"
+    joint_axis_xyz="0 0 1"
     visual_rpy="0 0 0"
     visual_xyz="0 0 0"
@@ -73,11 +68,8 @@
   />
   <!-- Front Castor Wheel -->
-  <joint name="caster_front_joint" type="fixed">
-    <parent link="base_link"/>
-    <child link="caster_front_link"/>
-    <origin xyz="0.115 0.0 0.007" rpy="${-M_PI/2} 0 0"/>
-  </joint>
-  <link_castor_kobuki
-    name="caster_front_link"
+  <castor_wheel_kobuki
+    name="caster_front"
+    joint_origin_xyz="0.115 0.0 0.007"
+    joint_origin_rpy="${-M_PI/2} 0 0"
     inertial_rpy="0 0 0"
     inertial_xyz="0 0 0"
@@ -91,11 +83,8 @@
   />
   <!-- Back Castor Wheel -->
-  <joint name="caster_back_joint" type="fixed">
-    <parent link="base_link"/>
-    <child link="caster_back_link"/>
-    <origin xyz="-0.135 0.0 0.009" rpy="${-M_PI/2} 0 0"/>
-  </joint>
-  <link_castor_kobuki
-    name="caster_back_link"
+  <castor_wheel_kobuki
+    name="caster_back"
+    joint_origin_xyz="-0.135 0.0 0.009"
+    joint_origin_rpy="${-M_PI/2} 0 0"
     inertial_rpy="0 0 0"
     inertial_xyz="0 0 0"
@@ -108,3 +97,12 @@
     iyy="0.001" iyz="0.0" izz="0.001"
   />
+  <!-- ******************************************************************************* -->
+  <!-- ******************************************************************************* -->
+  <!-- Gazebo Plugins -->
+  <gazebo>
+    <plugin name="gazebo_ros_control" filename="libgazebo_ros_control.so">
+      <robotNamespace>$(arg robot_namespace)</robotNamespace>
+      <legacyModeNS>true</legacyModeNS>
+    </plugin>
+  </gazebo>
 </robot>

File: urdf/kobuki_parameters.urdf.xacro (robot description, xacro)
@@ -34,9 +34,17 @@
     <!-- Traction Wheels Link Macro -->
     <xacro:macro
-    name="link_wheel_kobuki"
-    params="name visual_rpy visual_xyz inertial_xyz inertial_rpy
+    name="wheel_kobuki"
+    params="name
+            joint_origin_xyz joint_origin_rpy joint_axis_xyz
+            visual_rpy visual_xyz inertial_xyz inertial_rpy
             collision_xyz collision_rpy meshfile
             mass ixx ixy ixz iyy iyz izz cylinder_length cylinder_radius">
-        <link name="${name}">
+        <joint name="${name}_joint" type="continuous">
+            <parent link="base_link"/>
+            <child link="${name}_link"/>
+            <origin xyz="${joint_origin_xyz}" rpy="${joint_origin_rpy}"/>
+            <axis xyz="${joint_axis_xyz}"/>
+        </joint>
+        <link name="${name}_link">
             <visual>
                 <origin rpy="${visual_rpy}" xyz="${visual_xyz}" />
@@ -58,31 +66,34 @@
             </collision>
         </link>
-        <!-- <gazebo reference="${wheel_prefix}_wheel_link">
+        <!-- Friction values -->
+        <!-- Cambiar valores de mu1, mu2, fdir1 -->
+        <gazebo reference="${name}_link">
 			<mu1>0.01</mu1>
             <mu2>1</mu2>
             <fdir1>0 0 1</fdir1>
 		</gazebo>
-		<joint name="${wheel_prefix}_wheel" type="continuous">
-			<parent link="base_link"/>
-			<child link="${wheel_prefix}_wheel_link"/>
-			<xacro:insert_block name="joint_pose"/>
-			<axis xyz="0 1 0" rpy="0 0 0" />
-		</joint>
-		<transmission name="${wheel_prefix}_wheel_trans" type="SimpleTransmission">
-			<type>transmission_interface/SimpleTransmission</type>
-			<actuator name="${wheel_prefix}_wheel_motor">
-				<mechanicalReduction>1</mechanicalReduction>
-			</actuator>
-			<joint name="${wheel_prefix}_wheel">
-				<hardwareInterface>hardware_interface/VelocityJointInterface</hardwareInterface>
-			</joint>
-        </transmission> -->
+		<transmission name="${name}_tranmission">
+            <type>transmission_interface/SimpleTransmission</type>
+            <joint name="${name}_joint">
+                <hardwareInterface>hardware_interface/VelocityJointInterface</hardwareInterface>
+            </joint>
+            <actuator name="${name}_actuator">
+                <mechanicalReduction>1</mechanicalReduction>
+            </actuator>
+         </transmission>
     </xacro:macro>
     <!-- Castor Wheels Link Macro -->
     <xacro:macro
-    name="link_castor_kobuki"
-    params="name inertial_xyz inertial_rpy collision_xyz collision_rpy
+    name="castor_wheel_kobuki"
+    params="name
+            joint_origin_xyz joint_origin_rpy
+            inertial_xyz inertial_rpy collision_xyz collision_rpy
             mass ixx ixy ixz iyy iyz izz cylinder_length cylinder_radius">
-        <link name="${name}">
+        <joint name="${name}_joint" type="fixed">
+            <parent link="base_link"/>
+            <child link="${name}_link"/>
+            <origin xyz="${joint_origin_xyz}" rpy="${joint_origin_rpy}"/>
+        </joint>
+        <link name="${name}_link">
             <inertial>
                 <mass value="${mass}" />

Commit message: Cambios en scripts de python y algunas constantes de archivos xacro

File: urdf/kobuki_description.urdf.xacro (robot description, xacro)
@@ -14,4 +14,6 @@
   </joint>
   <!-- Base Link -->
+  <!-- ixx="0.019995" ixy="0.0" ixz="0.0" -->
+    <!-- iyy="0.019995" iyz="0.0" izz="0.03675"	 -->
   <link_base_kobuki
     name="base_link"
@@ -24,8 +26,8 @@
     cylinder_length="0.10938"
     cylinder_radius="0.178"
-    meshfile="package://kobuki_pkg/meshes/body.dae"
+    meshfile="package://kobuki_pkg/meshes/main_body.dae"
     mass="2.4"
-    ixx="0.019995" ixy="0.0" ixz="0.0"
-    iyy="0.019995" iyz="0.0" izz="0.03675"
+    ixx="0.021403" ixy="0.0" ixz="0.0"
+    iyy="0.021403" iyz="0.0" izz="0.038020"
   />
   <!-- Left Traction Wheel -->
@@ -45,6 +47,6 @@
     meshfile="package://kobuki_pkg/meshes/wheel.dae"
     mass="0.01"
-    ixx="0.001" ixy="0.0" ixz="0.0"
-    iyy="0.001" iyz="0.0" izz="0.001"
+    ixx="0.000892" ixy="0.0" ixz="0.0"
+    iyy="0.000892" iyz="0.0" izz="0.001584"
   />
   <!-- Right Traction Wheel -->
@@ -61,5 +63,5 @@
     collision_xyz="0 0 0"
     cylinder_length="0.0206"
-    cylinder_radius="0.035"
+    cylinder_radius="0.037"
     meshfile="package://kobuki_pkg/meshes/wheel.dae"
     mass="0.01"

File: urdf/kobuki_parameters.urdf.xacro (robot description, xacro)
@@ -62,5 +62,6 @@
                 <origin rpy="${collision_rpy}" xyz="${collision_xyz}" />
                 <geometry>
-                    <cylinder length="${cylinder_length}" radius="${cylinder_radius}"/>
+                    <!-- <cylinder length="${cylinder_length}" radius="${cylinder_radius}"/> -->
+                    <sphere radius="${cylinder_radius}"/>
                 </geometry>
             </collision>
@@ -104,5 +105,6 @@
                 <origin rpy="${collision_rpy}" xyz="${collision_xyz}" />
                 <geometry>
-                    <cylinder length="${cylinder_length}" radius="${cylinder_radius}"/>
+                    <!-- <cylinder length="${cylinder_length}" radius="${cylinder_radius}"/> -->
+                    <sphere radius="${cylinder_radius}"/>
                 </geometry>
             </collision>
